Commit message: we'll see

File: src/jaskier_urdf/urdf/jaskier.xacro (robot description, xacro)
@@ -7,5 +7,5 @@
     <xacro:property name="thumb_proximal" value="0.034"/>
     <xacro:property name="thumb_distal" value="0.032"/>
-    <xacro:property name="thumb_radius" value="0.017"/>
+    <xacro:property name="thumb_radius" value="0.0085"/>
     <xacro:property name="thumb_o_x" value="-${base_x/2}"/>
     <xacro:property name="thumb_o_y" value="-${base_y/2}"/>
@@ -29,5 +29,5 @@
     <xacro:property name="index_middle" value="0.024"/>
     <xacro:property name="index_distal" value="0.026"/>
-    <xacro:property name="index_radius" value="0.013"/>
+    <xacro:property name="index_radius" value="0.0065"/>
     <xacro:property name="index_o_x" value="-${base_x/2}"/>
     <xacro:property name="index_o_y" value="${base_y/2}"/>
@@ -54,5 +54,5 @@
     <xacro:property name="middle_middle" value="0.027"/>
     <xacro:property name="middle_distal" value="0.027"/>
-    <xacro:property name="middle_radius" value="0.014"/>
+    <xacro:property name="middle_radius" value="0.007"/>
 	<xacro:property name="middle_o_x" value="-${base_x/6}"/>
     <xacro:property name="middle_o_y" value="${base_y/2}"/>
@@ -79,5 +79,5 @@
     <xacro:property name="ring_middle" value="0.024"/>
     <xacro:property name="ring_distal" value="0.027"/>
-    <xacro:property name="ring_radius" value="0.013"/>
+    <xacro:property name="ring_radius" value="0.0065"/>
     <xacro:property name="ring_o_x" value="${base_x/6}"/>
     <xacro:property name="ring_o_y" value="${base_y/2}"/>
@@ -104,5 +104,5 @@
     <xacro:property name="little_middle" value="0.017"/>
     <xacro:property name="little_distal" value="0.025"/>
-    <xacro:property name="little_radius" value="0.012"/>
+    <xacro:property name="little_radius" value="0.006"/>
     <xacro:property name="little_o_x" value="${base_x/2}"/>
     <xacro:property name="little_o_y" value="${base_y/2}"/>
@@ -153,5 +153,5 @@
         <visual>
             <geometry>
-                <cyilnder length="${thumb_proximal}" radius="{thumb_radius}"/>
+                <cylinder length="${thumb_proximal}" radius="{thumb_radius}"/>
             </geometry>
             <xacro:thumb_proximal_vis/>
@@ -177,5 +177,5 @@
         <visual>
             <geometry>
-                <cyilnder length="${index_proximal}" radius="{index_radius}"/>
+                <cylinder length="${index_proximal}" radius="{index_radius}"/>
             </geometry>
             <xacro:index_proximal_vis/>
@@ -186,5 +186,5 @@
         <visual>
             <geometry>
-                <cyilnder length="${index_middle}" radius="{index_radius}"/>
+                <cylinder length="${index_middle}" radius="{index_radius}"/>
             </geometry>
             <xacro:index_middle_vis/>
@@ -210,5 +210,5 @@
         <visual>
             <geometry>
-                <cyilnder length="${middle_proximal}" radius="{middle_radius}"/>
+                <cylinder length="${middle_proximal}" radius="{middle_radius}"/>
             </geometry>
             <xacro:middle_proximal_vis/>
@@ -219,5 +219,5 @@
         <visual>
             <geometry>
-                <cyilnder length="${middle_middle}" radius="{middle_radius}"/>
+                <cylinder length="${middle_middle}" radius="{middle_radius}"/>
             </geometry>
             <xacro:middle_middle_vis/>
@@ -243,5 +243,5 @@
         <visual>
             <geometry>
-                <cyilnder length="${ring_proximal}" radius="{ring_radius}"/>
+                <cylinder length="${ring_proximal}" radius="{ring_radius}"/>
             </geometry>
             <xacro:ring_proximal_vis/>
@@ -252,5 +252,5 @@
         <visual>
             <geometry>
-                <cyilnder length="${ring_middle}" radius="{ring_radius}"/>
+                <cylinder length="${ring_middle}" radius="{ring_radius}"/>
             </geometry>
             <xacro:ring_middle_vis/>
@@ -276,5 +276,5 @@
         <visual>
             <geometry>
-                <cyilnder length="${little_proximal}" radius="{little_radius}"/>
+                <cylinder length="${little_proximal}" radius="{little_radius}"/>
             </geometry>
             <xacro:little_proximal_vis/>
@@ -285,5 +285,5 @@
         <visual>
             <geometry>
-                <cyilnder length="${little_middle}" radius="{little_radius}"/>
+                <cylinder length="${little_middle}" radius="{little_radius}"/>
             </geometry>
             <xacro:little_middle_vis/>

File: src/jaskier_urdf/urdf/jaskier_temp.urdf (robot description, URDF)
Before this commit: robot jaskier, 16 links, 15 joints
Links:
- link index_distal: geometry collision sphere radius=0.0065; visual cylinder length=0.026 radius=0.0065
- link index_middle: geometry visual cylinder length=0.024 radius={index_radius}
- link index_proximal: geometry visual cylinder length=0.026 radius={index_radius}
- link little_distal: geometry collision sphere radius=0.006; visual cylinder length=0.025 radius=0.006
- link little_middle: geometry visual cylinder length=0.017 radius={little_radius}
- link little_proximal: geometry visual cylinder length=0.018 radius={little_radius}
- link middle_distal: geometry collision sphere radius=0.007; visual cylinder length=0.027 radius=0.007
- link middle_middle: geometry visual cylinder length=0.027 radius={middle_radius}
- link middle_proximal: geometry visual cylinder length=0.026 radius={middle_radius}
- link ring_distal: geometry collision sphere radius=0.0065; visual cylinder length=0.027 radius=0.0065
- link ring_middle: geometry visual cylinder length=0.024 radius={ring_radius}
- link ring_proximal: geometry visual cylinder length=0.026 radius={ring_radius}
- link thumb_distal: geometry collision sphere radius=0.0085; visual cylinder length=0.032 radius=0.0085
- link thumb_proximal: geometry visual cylinder length=0.034 radius={thumb_radius}

Commit message: fixed xacro property references

File: src/jaskier_urdf/urdf/jaskier.xacro (robot description, xacro)
@@ -153,5 +153,5 @@
         <visual>
             <geometry>
-                <cylinder length="${thumb_proximal}" radius="{thumb_radius}"/>
+                <cylinder length="${thumb_proximal}" radius="${thumb_radius}"/>
             </geometry>
             <xacro:thumb_proximal_vis/>
@@ -177,5 +177,5 @@
         <visual>
             <geometry>
-                <cylinder length="${index_proximal}" radius="{index_radius}"/>
+                <cylinder length="${index_proximal}" radius="${index_radius}"/>
             </geometry>
             <xacro:index_proximal_vis/>
@@ -186,5 +186,5 @@
         <visual>
             <geometry>
-                <cylinder length="${index_middle}" radius="{index_radius}"/>
+                <cylinder length="${index_middle}" radius="${index_radius}"/>
             </geometry>
             <xacro:index_middle_vis/>
@@ -210,5 +210,5 @@
         <visual>
             <geometry>
-                <cylinder length="${middle_proximal}" radius="{middle_radius}"/>
+                <cylinder length="${middle_proximal}" radius="${middle_radius}"/>
             </geometry>
             <xacro:middle_proximal_vis/>
@@ -219,5 +219,5 @@
         <visual>
             <geometry>
-                <cylinder length="${middle_middle}" radius="{middle_radius}"/>
+                <cylinder length="${middle_middle}" radius="${middle_radius}"/>
             </geometry>
             <xacro:middle_middle_vis/>
@@ -243,5 +243,5 @@
         <visual>
             <geometry>
-                <cylinder length="${ring_proximal}" radius="{ring_radius}"/>
+                <cylinder length="${ring_proximal}" radius="${ring_radius}"/>
             </geometry>
             <xacro:ring_proximal_vis/>
@@ -276,5 +276,5 @@
         <visual>
             <geometry>
-                <cylinder length="${little_proximal}" radius="{little_radius}"/>
+                <cylinder length="${little_proximal}" radius="${little_radius}"/>
             </geometry>
             <xacro:little_proximal_vis/>
@@ -285,5 +285,5 @@
         <visual>
             <geometry>
-                <cylinder length="${little_middle}" radius="{little_radius}"/>
+                <cylinder length="${little_middle}" radius="${little_radius}"/>
             </geometry>
             <xacro:little_middle_vis/>

File: src/jaskier_urdf/urdf/jaskier_temp.urdf (robot description, URDF)
Before this commit: robot jaskier, 16 links, 15 joints
Links:
- link index_middle: geometry visual cylinder length=0.024 radius=0.0065
- link index_proximal: geometry visual cylinder length=0.026 radius=0.0065
- link little_middle: geometry visual cylinder length=0.017 radius=0.006
- link little_proximal: geometry visual cylinder length=0.018 radius=0.006
- link middle_middle: geometry visual cylinder length=0.027 radius=0.007
- link middle_proximal: geometry visual cylinder length=0.026 radius=0.007
- link ring_proximal: geometry visual cylinder length=0.026 radius=0.0065
- link thumb_proximal: geometry visual cylinder length=0.034 radius=0.0085

Commit message: missed one lol

File: src/jaskier_urdf/urdf/jaskier.xacro (robot description, xacro)
@@ -252,5 +252,5 @@
         <visual>
             <geometry>
-                <cylinder length="${ring_middle}" radius="{ring_radius}"/>
+                <cylinder length="${ring_middle}" radius="${ring_radius}"/>
             </geometry>
             <xacro:ring_middle_vis/>

File: src/jaskier_urdf/urdf/jaskier_temp.urdf (robot description, URDF)
Before this commit: robot jaskier, 16 links, 15 joints
Links:
- link ring_middle: geometry visual cylinder length=0.024 radius=0.0065

Commit message: fixed joint origin positions

File: src/jaskier_urdf/urdf/jaskier.xacro (robot description, xacro)
@@ -131,9 +131,6 @@
         </material>
     </xacro:macro>
-    <xacro:macro name="hand_digit_axis">
+    <xacro:macro name="joint_axis">
         <axis xyz="1 0 0"/>
-    </xacro:macro>
-    <xacro:macro name="digit_digit_axis">
-        <axis xyz="0 0 1"/>
     </xacro:macro>
     <xacro:macro name="joint_limit">
@@ -321,5 +318,5 @@
         <parent link="thumb_proximal"/>
         <child link="thumb_distal"/>
-        <xacro:digit_digit_axis/>
+        <xacro:joint_axis/>
         <xacro:joint_limit/>
         <origin xyz="0 0 ${thumb_proximal}" rpy="0 0 0"/>
@@ -328,5 +325,5 @@
         <parent link="hand_link"/>
         <child link="index_proximal"/>
-        <xacro:hand_digit_axis/>
+        <xacro:joint_axis/>
         <xacro:joint_limit/>
         <xacro:index_o/>
@@ -335,19 +332,19 @@
         <parent link="index_proximal"/>
         <child link="index_middle"/>
-        <xacro:digit_digit_axis/>
-        <xacro:joint_limit/>
-        <origin xyz="0 0 ${index_proximal}" rpy="0 0 0"/>
+        <xacro:joint_axis/>
+        <xacro:joint_limit/>
+        <origin xyz="0 0 -${index_proximal}" rpy="0 0 0"/>
     </joint>
     <joint name="index_dip" type="revolute">
         <parent link="index_middle"/>
         <child link="index_distal"/>
-        <xacro:digit_digit_axis/>
-        <xacro:joint_limit/>
-        <origin xyz="0 0 ${index_middle}" rpy="0 0 0"/>
+        <xacro:joint_axis/>
+        <xacro:joint_limit/>
+        <origin xyz="0 0 -${index_middle}" rpy="0 0 0"/>
     </joint>
     <joint name="middle_mcp" type="revolute">
         <parent link="hand_link"/>
         <child link="middle_proximal"/>
-        <xacro:hand_digit_axis/>
+        <xacro:joint_axis/>
         <xacro:joint_limit/>
         <xacro:middle_o/>
@@ -356,19 +353,19 @@
         <parent link="middle_proximal"/>
         <child link="middle_middle"/>
-        <xacro:digit_digit_axis/>
-        <xacro:joint_limit/>
-        <origin xyz="0 0 ${middle_proximal}" rpy="0 0 0"/>
+        <xacro:joint_axis/>
+        <xacro:joint_limit/>
+        <origin xyz="0 0 -${middle_proximal}" rpy="0 0 0"/>
     </joint>
     <joint name="middle_dip" type="revolute">
         <parent link="middle_middle"/>
         <child link="middle_distal"/>
-        <xacro:digit_digit_axis/>
-        <xacro:joint_limit/>
-        <origin xyz="0 0 ${middle_middle}" rpy="0 0 0"/>
+        <xacro:joint_axis/>
+        <xacro:joint_limit/>
+        <origin xyz="0 0 -${middle_middle}" rpy="0 0 0"/>
     </joint>
     <joint name="ring_mcp" type="revolute">
         <parent link="hand_link"/>
         <child link="ring_proximal"/>
-        <xacro:hand_digit_axis/>
+        <xacro:joint_axis/>
         <xacro:joint_limit/>
         <xacro:ring_o/>
@@ -377,19 +374,19 @@
         <parent link="ring_proximal"/>
         <child link="ring_middle"/>
-        <xacro:digit_digit_axis/>
-        <xacro:joint_limit/>
-        <origin xyz="0 0 ${ring_proximal}" rpy="0 0 0"/>
+        <xacro:joint_axis/>
+        <xacro:joint_limit/>
+        <origin xyz="0 0 -${ring_proximal}" rpy="0 0 0"/>
     </joint>
     <joint name="ring_dip" type="revolute">
         <parent link="ring_middle"/>
         <child link="ring_distal"/>
-        <xacro:digit_digit_axis/>
-        <xacro:joint_limit/>
-        <origin xyz="0 0 ${ring_middle}" rpy="0 0 0"/>
+        <xacro:joint_axis/>
+        <xacro:joint_limit/>
+        <origin xyz="0 0 -${ring_middle}" rpy="0 0 0"/>
     </joint>
     <joint name="little_mcp" type="revolute">
         <parent link="hand_link"/>
         <child link="little_proximal"/>
-        <xacro:hand_digit_axis/>
+        <xacro:joint_axis/>
         <xacro:joint_limit/>
         <xacro:little_o/>
@@ -398,14 +395,14 @@
         <parent link="little_proximal"/>
         <child link="little_middle"/>
-        <xacro:digit_digit_axis/>
-        <xacro:joint_limit/>
-        <origin xyz="0 0 ${little_proximal}" rpy="0 0 0"/>
+        <xacro:joint_axis/>
+        <xacro:joint_limit/>
+        <origin xyz="0 0 -${little_proximal}" rpy="0 0 0"/>
     </joint>
     <joint name="little_dip" type="revolute">
         <parent link="little_middle"/>
         <child link="little_distal"/>
-        <xacro:digit_digit_axis/>
-        <xacro:joint_limit/>
-        <origin xyz="0 0 ${little_middle}" rpy="0 0 0"/>
+        <xacro:joint_axis/>
+        <xacro:joint_limit/>
+        <origin xyz="0 0 -${little_middle}" rpy="0 0 0"/>
     </joint>
 </robot>

File: src/jaskier_urdf/urdf/jaskier_temp.urdf (robot description, URDF)
Before this commit: robot jaskier, 16 links, 15 joints
Joints:
- joint index_dip: axis 0 0 1 -> 1 0 0; origin xyz=0 0 0.024 rpy=0 0 0 -> xyz=0 0 -0.024 rpy=0 0 0
- joint index_pip: axis 0 0 1 -> 1 0 0; origin xyz=0 0 0.026 rpy=0 0 0 -> xyz=0 0 -0.026 rpy=0 0 0
- joint little_dip: axis 0 0 1 -> 1 0 0; origin xyz=0 0 0.017 rpy=0 0 0 -> xyz=0 0 -0.017 rpy=0 0 0
- joint little_pip: axis 0 0 1 -> 1 0 0; origin xyz=0 0 0.018 rpy=0 0 0 -> xyz=0 0 -0.018 rpy=0 0 0
- joint middle_dip: axis 0 0 1 -> 1 0 0; origin xyz=0 0 0.027 rpy=0 0 0 -> xyz=0 0 -0.027 rpy=0 0 0
- joint middle_pip: axis 0 0 1 -> 1 0 0; origin xyz=0 0 0.026 rpy=0 0 0 -> xyz=0 0 -0.026 rpy=0 0 0
- joint ring_dip: axis 0 0 1 -> 1 0 0; origin xyz=0 0 0.024 rpy=0 0 0 -> xyz=0 0 -0.024 rpy=0 0 0
- joint ring_pip: axis 0 0 1 -> 1 0 0; origin xyz=0 0 0.026 rpy=0 0 0 -> xyz=0 0 -0.026 rpy=0 0 0
- joint thumb_ip: axis 0 0 1 -> 1 0 0

Commit message: fixed thumb

File: src/jaskier_urdf/urdf/jaskier.xacro (robot description, xacro)
@@ -12,5 +12,5 @@
     <xacro:property name="thumb_o_r" value="0.9"/>
     <xacro:property name="thumb_o_p" value="0.6"/>
-    <xacro:property name="thumb_o_xyz" value="${thumb_o_x} ${thumb_o_y} 0"/>
+    <xacro:property name="thumb_o_xyz" value="${thumb_o_x} ${thumb_o_y} -${base_z}"/>
     <xacro:property name="thumb_o_rpy" value="${thumb_o_r} ${thumb_o_p} 0"/>
     <xacro:macro name="thumb_o">
@@ -318,7 +318,7 @@
         <parent link="thumb_proximal"/>
         <child link="thumb_distal"/>
-        <xacro:joint_axis/>
-        <xacro:joint_limit/>
-        <origin xyz="0 0 ${thumb_proximal}" rpy="0 0 0"/>
+        <axis xyz="0 1 0"/>
+        <xacro:joint_limit/>
+        <origin xyz="0 0 -${thumb_proximal}" rpy="0 0 0"/>
     </joint>
     <joint name="index_mcp" type="revolute">

File: src/jaskier_urdf/urdf/jaskier_temp.urdf (robot description, URDF)
Before this commit: robot jaskier, 16 links, 15 joints
Joints:
- joint thumb_ip: axis 1 0 0 -> 0 1 0; origin xyz=0 0 0.034 rpy=0 0 0 -> xyz=0 0 -0.034 rpy=0 0 0
- joint thumb_mcp: origin xyz=-0.0425 -0.0305 0 rpy=0.9 0.6 0 -> xyz=-0.0425 -0.0305 -0.02 rpy=0.9 0.6 0
