Commit message: linked jaskier model to adc

File: src/jaskier_urdf/urdf/jaskier.urdf (robot description, URDF)
Before this commit: robot jaskier, 6 links, 5 joints
Joints:
- joint index_joint: axis 0 1 0 -> 1 0 0; limit lower=0.0 upper=1.8 effort=0.0 velocity=20 -> lower=-1.8 upper=0 effort=0.0 velocity=20; origin xyz=-0.04 0.04 0 rpy=0 0 0 -> xyz=-0.04 0.04 0 rpy=1.57079632679 0 0
- joint little_joint: axis 0 1 0 -> 1 0 0; limit lower=0.0 upper=1.8 effort=0.0 velocity=20 -> lower=-1.8 upper=0 effort=0.0 velocity=20; origin xyz=0.04 0.04 0 rpy=0 0 0 -> xyz=0.04 0.04 0 rpy=1.57079632679 0 0
- joint middle_joint: axis 0 1 0 -> 1 0 0; limit lower=0.0 upper=1.8 effort=0.0 velocity=20 -> lower=-1.8 upper=0 effort=0.0 velocity=20; origin xyz=-0.0133333333333 0.04 0 rpy=0 0 0 -> xyz=-0.0133333333333 0.04 0 rpy=1.57079632679 0 0
- joint ring_joint: axis 0 1 0 -> 1 0 0; limit lower=0.0 upper=1.8 effort=0.0 velocity=20 -> lower=-1.8 upper=0 effort=0.0 velocity=20; origin xyz=0.0133333333333 0.04 0 rpy=0 0 0 -> xyz=0.0133333333333 0.04 0 rpy=1.57079632679 0 0
- joint thumb_joint: limit lower=0.0 upper=1.8 effort=0.0 velocity=20 -> lower=-1.8 upper=0 effort=0.0 velocity=20; origin xyz=-0.04 -0.04 0 rpy=-1.57079632679 0.785398163397 0 -> xyz=-0.04 -0.04 0 rpy=0.9 0.6 0

Commit message: collision module initial work

File: src/jaskier_urdf/urdf/jaskier.urdf (robot description, URDF)
Before this commit: robot jaskier, 6 links, 5 joints
Links:
- removed link base_link
- added link hand_link; visual box size=0.08 0.08 0.02
Joints:
- joint index_joint: parent base_link -> hand_link
- joint little_joint: parent base_link -> hand_link
- joint middle_joint: parent base_link -> hand_link
- joint ring_joint: parent base_link -> hand_link
- joint thumb_joint: parent base_link -> hand_link

File: src/jaskier_urdf/urdf/jaskier.xacro (robot description, xacro)
@@ -97,5 +97,5 @@
         <limit effort="0.0" velocity="20" lower="-1.8" upper="0"/>
     </xacro:macro>
-    <link name="base_link">
+    <link name="hand_link">
         <visual>
             <geometry>
@@ -183,5 +183,5 @@
     </link>
     <joint name="thumb_joint" type="revolute">
-        <parent link="base_link"/>
+        <parent link="hand_link"/>
         <child link="thumb"/>
         <axis xyz="0 1 0"/>
@@ -190,5 +190,5 @@
     </joint>
     <joint name="index_joint" type="revolute">
-        <parent link="base_link"/>
+        <parent link="hand_link"/>
         <child link="index"/>
         <xacro:joint_axis/>
@@ -197,5 +197,5 @@
     </joint>
     <joint name="middle_joint" type="revolute">
-        <parent link="base_link"/>
+        <parent link="hand_link"/>
         <child link="middle"/>
         <xacro:joint_axis/>
@@ -204,5 +204,5 @@
     </joint>
     <joint name="ring_joint" type="revolute">
-        <parent link="base_link"/>
+        <parent link="hand_link"/>
         <child link="ring"/>
         <xacro:joint_axis/>
@@ -211,5 +211,5 @@
     </joint>
     <joint name="little_joint" type="revolute">
-        <parent link="base_link"/>
+        <parent link="hand_link"/>
         <child link="little"/>
         <xacro:joint_axis/>

Commit message: updated hand model

File: src/jaskier_urdf/urdf/jaskier.urdf (robot description, URDF)
Before this commit: robot jaskier, 6 links, 5 joints
Links:
- removed link index
- removed link little
- removed link middle
- removed link ring
- removed link thumb
- added link imu
- added link index_distal; collision sphere radius=0.0065; visual cylinder length=0.026 radius=0.0065
- added link index_middle; visual cylinder length=0.024 radius=0.0065
- added link index_proximal; visual cylinder length=0.026 radius=0.0065
- added link little_distal; collision sphere radius=0.006; visual cylinder length=0.025 radius=0.006
- added link little_middle; visual cylinder length=0.017 radius=0.006
- added link little_proximal; visual cylinder length=0.018 radius=0.006
- added link middle_distal; collision sphere radius=0.007; visual cylinder length=0.027 radius=0.007
- added link middle_middle; visual cylinder length=0.027 radius=0.007
- added link middle_proximal; visual cylinder length=0.026 radius=0.007
- added link ring_distal; collision sphere radius=0.0065; visual cylinder length=0.027 radius=0.0065
- added link ring_middle; visual cylinder length=0.024 radius=0.0065
- added link ring_proximal; visual cylinder length=0.026 radius=0.0065
- added link thumb_distal; collision sphere radius=0.0085; visual cylinder length=0.032 radius=0.0085
- added link thumb_proximal; visual cylinder length=0.034 radius=0.0085
- link hand_link: geometry visual box size=0.085 0.061 0.02
Joints:
- removed joint index_joint
- removed joint little_joint
- removed joint middle_joint
- removed joint ring_joint
- removed joint thumb_joint
- added joint imu_joint: type floating, parent imu, child hand_link
- added joint index_dip: type revolute, parent index_middle, child index_distal, origin xyz=0 0 -0.024 rpy=0 0 0, axis 1 0 0, limit lower=-1.8 upper=0 effort=0.0 velocity=20
- added joint index_mcp: type revolute, parent hand_link, child index_proximal, origin xyz=-0.0425 0.0305 0 rpy=1.57079632679 0 0, axis 1 0 0, limit lower=-1.8 upper=0 effort=0.0 velocity=20
- added joint index_pip: type revolute, parent index_proximal, child index_middle, origin xyz=0 0 -0.026 rpy=0 0 0, axis 1 0 0, limit lower=-1.8 upper=0 effort=0.0 velocity=20
- added joint little_dip: type revolute, parent little_middle, child little_distal, origin xyz=0 0 -0.017 rpy=0 0 0, axis 1 0 0, limit lower=-1.8 upper=0 effort=0.0 velocity=20
- added joint little_mcp: type revolute, parent hand_link, child little_proximal, origin xyz=0.0425 0.0305 0 rpy=1.57079632679 0 0, axis 1 0 0, limit lower=-1.8 upper=0 effort=0.0 velocity=20
- added joint little_pip: type revolute, parent little_proximal, child little_middle, origin xyz=0 0 -0.018 rpy=0 0 0, axis 1 0 0, limit lower=-1.8 upper=0 effort=0.0 velocity=20
- added joint middle_dip: type revolute, parent middle_middle, child middle_distal, origin xyz=0 0 -0.027 rpy=0 0 0, axis 1 0 0, limit lower=-1.8 upper=0 effort=0.0 velocity=20
- added joint middle_mcp: type revolute, parent hand_link, child middle_proximal, origin xyz=-0.0141666666667 0.0305 0 rpy=1.57079632679 0 0, axis 1 0 0, limit lower=-1.8 upper=0 effort=0.0 velocity=20
- added joint middle_pip: type revolute, parent middle_proximal, child middle_middle, origin xyz=0 0 -0.026 rpy=0 0 0, axis 1 0 0, limit lower=-1.8 upper=0 effort=0.0 velocity=20
- added joint ring_dip: type revolute, parent ring_middle, child ring_distal, origin xyz=0 0 -0.024 rpy=0 0 0, axis 1 0 0, limit lower=-1.8 upper=0 effort=0.0 velocity=20
- added joint ring_mcp: type revolute, parent hand_link, child ring_proximal, origin xyz=0.0141666666667 0.0305 0 rpy=1.57079632679 0 0, axis 1 0 0, limit lower=-1.8 upper=0 effort=0.0 velocity=20
- added joint ring_pip: type revolute, parent ring_proximal, child ring_middle, origin xyz=0 0 -0.026 rpy=0 0 0, axis 1 0 0, limit lower=-1.8 upper=0 effort=0.0 velocity=20
- added joint thumb_ip: type revolute, parent thumb_proximal, child thumb_distal, origin xyz=0 0 -0.034 rpy=0 0 0, axis 0 1 0, limit lower=-1.8 upper=0 effort=0.0 velocity=20
- added joint thumb_mcp: type revolute, parent hand_link, child thumb_proximal, origin xyz=-0.0425 -0.0305 -0.02 rpy=0.9 0.6 0, axis 0 1 0, limit lower=-1.8 upper=0 effort=0.0 velocity=20

Commit message: added imu and ultrasonic joints

File: src/jaskier_urdf/urdf/jaskier.urdf (robot description, URDF)
Before this commit: robot jaskier, 16 links, 15 joints
Links:
- removed link imu
- added link base_link
- added link imu_x_link
- added link imu_y_link
- added link imu_z_link
- added link ultra_x_link
- added link ultra_y_link
- added link ultra_z_link
Joints:
- removed joint imu_joint
- added joint base_joint: type fixed, parent base_link, child ultra_z_link
- added joint imu_x: type continuous, parent imu_x_link, child hand_link, axis 1 0 0
- added joint imu_y: type continuous, parent imu_y_link, child imu_x_link, axis 0 1 0
- added joint imu_z: type continuous, parent imu_z_link, child imu_y_link, axis 0 0 1
- added joint ultra_x: type prismatic, parent ultra_x_link, child imu_z_link, axis 1 0 0
- added joint ultra_y: type prismatic, parent ultra_y_link, child ultra_x_link, axis 0 1 0
- added joint ultra_z: type prismatic, parent ultra_z_link, child ultra_y_link, axis 0 0 1

File: src/jaskier_urdf/urdf/jaskier.xacro (robot description, xacro)
@@ -303,8 +303,44 @@
         </collision>
     </link>
-    <link name="imu"/>
-    <joint name="imu_joint" type="floating">
-        <parent link="imu"/>
+    <link name="imu_x_link"/>
+    <link name="imu_y_link"/>
+    <link name="imu_z_link"/>
+    <link name="ultra_x_link"/>
+    <link name="ultra_y_link"/>
+    <link name="ultra_z_link"/>
+    <link name="base_link"/>
+    <joint name="imu_x" type="continuous">
+        <parent link="imu_x_link"/>
         <child link="hand_link"/>
+        <axis xyz="1 0 0"/>
+    </joint>
+    <joint name="imu_y" type="continuous">
+        <parent link="imu_y_link"/>
+        <child link="imu_x_link"/>
+        <axis xyz="0 1 0"/>
+    </joint>
+    <joint name="imu_z" type="continuous">
+        <parent link="imu_z_link"/>
+        <child link="imu_y_link"/>
+        <axis xyz="0 0 1"/>
+    </joint>
+    <joint name="ultra_x" type="prismatic">
+        <parent link="ultra_x_link"/>
+        <child link="imu_z_link"/>
+        <axis xyz="1 0 0"/>
+    </joint>
+    <joint name="ultra_y" type="prismatic">
+        <parent link="ultra_y_link"/>
+        <child link="ultra_x_link"/>
+        <axis xyz="0 1 0"/>
+    </joint>
+    <joint name="ultra_z" type="prismatic">
+        <parent link="ultra_z_link"/>
+        <child link="ultra_y_link"/>
+        <axis xyz="0 0 1"/>
+    </joint>
+    <joint name="base_joint" type="fixed">
+        <parent link="base_link"/>
+        <child link="ultra_z_link"/>
     </joint>
     <joint name="thumb_mcp" type="revolute">

Commit message: all hand sensors linked to model

File: src/jaskier_urdf/urdf/jaskier.urdf (robot description, URDF)
Before this commit: robot jaskier, 22 links, 21 joints
Joints:
- joint ultra_x: limit (none) -> lower=-20 upper=20 effort=0.0 velocity=20
- joint ultra_y: limit (none) -> lower=-20 upper=20 effort=0.0 velocity=20
- joint ultra_z: limit (none) -> lower=-20 upper=20 effort=0.0 velocity=20

File: src/jaskier_urdf/urdf/jaskier.xacro (robot description, xacro)
@@ -137,4 +137,7 @@
         <limit effort="0.0" velocity="20" lower="-1.8" upper="0"/>
     </xacro:macro>
+    <xacro:macro name="prismatic_limit">
+        <limit effort="0.0" velocity="20" lower="-20" upper="20"/>
+    </xacro:macro>
     <link name="hand_link">
         <visual>
@@ -329,4 +332,5 @@
         <child link="imu_z_link"/>
         <axis xyz="1 0 0"/>
+        <xacro:prismatic_limit/>
     </joint>
     <joint name="ultra_y" type="prismatic">
@@ -334,4 +338,5 @@
         <child link="ultra_x_link"/>
         <axis xyz="0 1 0"/>
+        <xacro:prismatic_limit/>
     </joint>
     <joint name="ultra_z" type="prismatic">
@@ -339,4 +344,5 @@
         <child link="ultra_y_link"/>
         <axis xyz="0 0 1"/>
+        <xacro:prismatic_limit/>
     </joint>
     <joint name="base_joint" type="fixed">
